File: board/board.kicad_pcb (KiCad board)
At the start: 2 copper layers, 21 x 13 mm, 1 part

Commit message: initial
Parts:
- added C1: 100nF, Capacitor_SMD:C_0603_1608Metric, F.Cu at (153.5, 100.0)
- added C2: 1uF, Capacitor_SMD:C_0603_1608Metric, F.Cu at (155.0, 100.0)
- added C3: 10uF, Capacitor_SMD:C_0603_1608Metric, F.Cu at (148.5, 98.2)
- added C4: 1uF, Capacitor_SMD:C_0603_1608Metric, F.Cu at (146.9, 98.2)
- added J1: 003_power, on_edge:on_edge_2x05_device, F.Cu at (140.0, 96.5)
- added J2: 003_power, on_edge:on_edge_2x05_host, F.Cu at (161.0, 96.5)
- added J3: Conn_01x03_Male, Connector_PinHeader_2.54mm:PinHeader_1x03_P2.54mm_Vertical, F.Cu at (146.1, 101.6)
- added R1: 0R, Resistor_SMD:R_0603_1608Metric, B.Cu at (146.5, 98.5)
- added R2: 0R, Resistor_SMD:R_0603_1608Metric, B.Cu at (151.1, 96.3)
- added U1: TLV743P, Package_TO_SOT_SMD:SOT-23-5, F.Cu at (151.0, 97.7)
- LOGO1: moved to B.Cu
- moved LOGO1 5.95 mm to (150.8, 93.1), turned to 180 degrees
Routing:
- net /ldo/GND: track 0.00 -> 38.6 mm, vias 0 -> 2
- net Net-(J1-Pad5): track 0.00 -> 21.4 mm
- net /ldo/5v: track 0.00 -> 20.9 mm, vias 0 -> 2
- net Net-(J1-Pad8): track 0.00 -> 20.0 mm
- net Net-(J1-Pad4): track 0.00 -> 19.7 mm
- net Net-(J1-Pad7): track 0.00 -> 19.4 mm
- net Net-(J1-Pad3): track 0.00 -> 18.6 mm
- net Net-(J1-Pad6): track 0.00 -> 17.9 mm
- net Net-(J1-Pad2): track 0.00 -> 15.8 mm
- net Net-(U1-Pad3): track 0.00 -> 8.12 mm, vias 0 -> 1
- net Net-(J2-Pad9): track 0.00 -> 7.59 mm
- net /ldo/3.3v: track 0.00 -> 7.56 mm, vias 0 -> 2
- net Net-(J1-Pad9): track 0.00 -> 3.28 mm
Other:
- outline, holes or cut-outs redrawn
- board text added: "enable"
- board text added: "osf.003"
- board text added: "osf.b103.v1.0"
